Commit message: Added industrial robot model

File: model/macros/inertia.xacro (robot description, xacro)
@@ -6,4 +6,12 @@
     iyy="${mass*(radius**2/4 + length**2/12)}"
     izz="${mass*(radius**2/2)}"
+    ixy="0" ixz="0" iyz="0"
+/>
+</xacro:macro>
+<xacro:macro name="box_inertia_urdf" params="mass w h d">
+<inertia
+    ixx="${mass*(h**2 + d**2)/12}"
+    iyy="${mass*(w**2 + d**2)/12}"
+    izz="${mass*(w**2 + h**2)/12}"
     ixy="0" ixz="0" iyz="0"
 />
