Commit message: Updated urdf to use mimic tags

File: model/delta/ros_joints/lower.urdf.xacro (robot description, xacro)
@@ -2,5 +2,5 @@
 <robot xmlns:xacro="http://www.ros.org/wiki/xacro" name="delta">
 <xacro:macro name="joints_lower" params="number">
-<joint name="lower_${number}_alpha" type="revolute">
+<joint name="alpha_${number}" type="revolute">
     <axis xyz="0 1 0"/>
     <limit effort="1000.0" lower="${-pi/2}" upper="${pi/2}" velocity="0.5"/>
@@ -15,5 +15,5 @@
 <link name="lower_${number}_root">
 </link>
-<joint name="lower_${number}_L_beta_top" type="revolute">
+<joint name="beta_${number}" type="revolute">
     <axis xyz="0 0 1"/>
     <limit effort="1000.0" lower="${-pi/2}" upper="${pi/2}" velocity="0.5"/>
@@ -25,5 +25,5 @@
     <child link="lower_${number}_L_link"/>
 </joint>
-<joint name="lower_${number}_L_beta_bot" type="revolute">
+<joint name="beta_${number}_L_bot" type="revolute">
     <axis xyz="0 0 1"/>
     <limit effort="1000.0" lower="${-pi/2}" upper="${pi/2}" velocity="0.5"/>
@@ -34,9 +34,10 @@
     <parent link="lower_${number}_L_link"/>
     <child link="lower_${number}_L_link_end"/>
+    <mimic joint="beta_${number}" multiplier="-1"/>
 </joint>
 <!-- Virtual link -->
 <link name="lower_${number}_L_link_end">
 </link>
-<joint name="lower_${number}_L_gamma" type="revolute">
+<joint name="gamma_${number}" type="revolute">
     <axis xyz="0 1 0"/>
     <limit effort="1000.0" lower="${-pi/2}" upper="${pi/2}" velocity="0.5"/>
@@ -59,5 +60,5 @@
     <child link="chain_${number}_end"/>
 </joint>
-<joint name="lower_${number}_R_beta_top" type="revolute">
+<joint name="beta_${number}_R_top" type="revolute">
     <axis xyz="0 0 1"/>
     <limit effort="1000.0" lower="${-pi/2}" upper="${pi/2}" velocity="0.5"/>
@@ -68,4 +69,5 @@
     <parent link="lower_${number}_root"/>
     <child link="lower_${number}_R_link"/>
+    <mimic joint="beta_${number}"/>
 </joint>
 <!-- Virtual link -->

Commit message: Tweaked some settings, in particular - joint velocity limits.

File: model/delta/ros_joints/lower.urdf.xacro (robot description, xacro)
@@ -4,5 +4,5 @@
 <joint name="alpha_${number}" type="revolute">
     <axis xyz="0 1 0"/>
-    <limit effort="1000.0" lower="${-pi/2}" upper="${pi/2}" velocity="0.5"/>
+    <limit effort="1000.0" lower="${-pi/2}" upper="${pi/2}" velocity="100"/>
     <origin
         rpy="0 0 0"
@@ -17,5 +17,5 @@
 <joint name="beta_${number}" type="revolute">
     <axis xyz="0 0 1"/>
-    <limit effort="1000.0" lower="${-pi/2}" upper="${pi/2}" velocity="0.5"/>
+    <limit effort="1000.0" lower="${-pi/2}" upper="${pi/2}" velocity="100"/>
     <origin
         rpy="0 0 0"
@@ -27,5 +27,5 @@
 <joint name="beta_${number}_L_bot" type="revolute">
     <axis xyz="0 0 1"/>
-    <limit effort="1000.0" lower="${-pi/2}" upper="${pi/2}" velocity="0.5"/>
+    <limit effort="1000.0" lower="${-pi/2}" upper="${pi/2}" velocity="100"/>
     <origin
         rpy="0 0 0"
@@ -41,5 +41,5 @@
 <joint name="gamma_${number}" type="revolute">
     <axis xyz="0 1 0"/>
-    <limit effort="1000.0" lower="${-pi/2}" upper="${pi/2}" velocity="0.5"/>
+    <limit effort="1000.0" lower="${-pi/2}" upper="${pi/2}" velocity="100"/>
     <origin
         rpy="0 0 0"
@@ -62,5 +62,5 @@
 <joint name="beta_${number}_R_top" type="revolute">
     <axis xyz="0 0 1"/>
-    <limit effort="1000.0" lower="${-pi/2}" upper="${pi/2}" velocity="0.5"/>
+    <limit effort="1000.0" lower="${-pi/2}" upper="${pi/2}" velocity="100"/>
     <origin
         rpy="0 0 0"

File: model/delta/ros_joints/upper.urdf.xacro (robot description, xacro)
@@ -9,5 +9,5 @@
         lower="${-pi/2}"
         upper="${pi/2}"
-        velocity="0.5"
+        velocity="5"
     />
     <origin
