Commit message: Delta model works with gripper rotation now

File: model/delta/ros_joints/end_effector.urdf.xacro (robot description, xacro)
@@ -7,5 +7,5 @@
 </joint>
 <joint name="theta_4" type="revolute">
-    <origin xyz="0 0 0" rpy="0 0 0"/>
+    <origin xyz="0 0 0" rpy="0 0 ${-pi/3}"/>
     <parent link="ee"/>
     <child link="gripper_base"/>
@@ -13,6 +13,6 @@
     <limit
         effort="1000.0"
-        lower="${-pi*0.99}"
-        upper="${pi*0.99}"
+        lower="${-pi/2}"
+        upper="${pi/2}"
         velocity="5"
     />

File: model/delta/ros_links/end_effector.urdf.xacro (robot description, xacro)
@@ -66,5 +66,5 @@
         <box size="0.05 0.1 0.08"/>
     </geometry>
-    <origin xyz="0 0 -0.04"/>
+    <origin xyz="0 0 -0.04" rpy="0 0 0"/>
 </visual>
 <collision>
@@ -72,5 +72,5 @@
         <box size="0.05 0.1 0.08"/>
     </geometry>
-    <origin xyz="0 0 -0.04"/>
+    <origin xyz="0 0 -0.04" rpy="0 0 0"/>
 </collision>
 </link>

Commit message: Made delta gripper the correct size

File: model/delta/ros_joints/end_effector.urdf.xacro (robot description, xacro)
@@ -19,5 +19,5 @@
 </joint>
 <joint name="gripper" type="revolute">
-    <origin xyz="0 -0.05 -0.08" rpy="0.6 0 0"/>
+    <origin xyz="0 -0.025 -0.05" rpy="0.4 0 0"/>
     <parent link="gripper_base"/>
     <child link="gripper_left"/>
@@ -31,5 +31,5 @@
 </joint>
 <joint name="gripper_mimic" type="revolute">
-    <origin xyz="0 0.05 -0.08" rpy="-0.6 0 0"/>
+    <origin xyz="0 0.025 -0.05" rpy="-0.4 0 0"/>
     <parent link="gripper_base"/>
     <child link="gripper_right"/>

File: model/delta/ros_links/end_effector.urdf.xacro (robot description, xacro)
@@ -64,13 +64,13 @@
 <visual>
     <geometry>
-        <box size="0.05 0.1 0.08"/>
+        <box size="0.03 0.05 0.05"/>
     </geometry>
-    <origin xyz="0 0 -0.04" rpy="0 0 0"/>
+    <origin xyz="0 0 -0.025" rpy="0 0 0"/>
 </visual>
 <collision>
     <geometry>
-        <box size="0.05 0.1 0.08"/>
+        <box size="0.05 0.03 0.05"/>
     </geometry>
-    <origin xyz="0 0 -0.04" rpy="0 0 0"/>
+    <origin xyz="0 0 -0.025" rpy="0 0 0"/>
 </collision>
 </link>
@@ -78,13 +78,13 @@
 <visual>
     <geometry>
-        <box size="0.05 0.005 0.1"/>
+        <box size="0.03 0.005 0.05"/>
     </geometry>
-    <origin xyz="0 0 -0.05"/>
+    <origin xyz="0 0 -0.025"/>
 </visual>
 <collision>
     <geometry>
-        <box size="0.05 0.005 0.1"/>
+        <box size="0.03 0.005 0.05"/>
     </geometry>
-    <origin xyz="0 0 -0.05"/>
+    <origin xyz="0 0 -0.025"/>
 </collision>
 </link>
@@ -92,13 +92,13 @@
 <visual>
     <geometry>
-        <box size="0.05 0.005 0.1"/>
+        <box size="0.03 0.005 0.05"/>
     </geometry>
-    <origin xyz="0 0 -0.05"/>
+    <origin xyz="0 0 -0.025"/>
 </visual>
 <collision>
     <geometry>
-        <box size="0.05 0.005 0.1"/>
+        <box size="0.03 0.005 0.05"/>
     </geometry>
-    <origin xyz="0 0 -0.05"/>
+    <origin xyz="0 0 -0.025"/>
 </collision>
 </link>
