Commit message: Renamed some things. Commented out serial model gains since gazebo_ros_control not working.

File: model/serial/parameters.xacro (robot description, xacro)
@@ -17,10 +17,10 @@
 <xacro:property name="arm_radius" value="0.05"/>
 <xacro:property name="wrist_radius" value="0.03"/>
-<xacro:property name="fixed_base_mass" value="0.5"/>
-<xacro:property name="base_mass" value="0.5"/>
-<xacro:property name="lower_mass" value="0.1"/>
-<xacro:property name="upper_mass" value="0.1"/>
+<xacro:property name="fixed_base_mass" value="1"/>
+<xacro:property name="base_mass" value="1"/>
+<xacro:property name="lower_mass" value="0.5"/>
+<xacro:property name="upper_mass" value="0.5"/>
 <xacro:property name="wrist_roll_mass" value="0.1"/>
 <xacro:property name="wrist_pitch_mass" value="0.1"/>
-<xacro:property name="tool_base_mass" value="0.1"/>
+<xacro:property name="tool_base_mass" value="0.05"/>
 </robot>

File: model/serial/ros.urdf.xacro (robot description, xacro)
@@ -1,4 +1,4 @@
 <?xml version="1.0"?>
-<robot xmlns:xacro="http://www.ros.org/wiki/xacro" name="industrial">
+<robot xmlns:xacro="http://www.ros.org/wiki/xacro" name="serial">
 <xacro:include filename="../macros/inertia.xacro"/>
 <xacro:include filename="parameters.xacro"/>
