Commit message: Tidied up things

File: model/delta/gazebo_joints/end_effector.sdf.xacro (robot description, xacro)
@@ -1,28 +1,28 @@
 <?xml version="1.0"?>
 <robot xmlns:xacro="http://www.ros.org/wiki/xacro" name="delta">
-<xacro:macro name="joints_end_effector" params="number yaw">
+<xacro:macro name="joints_ee" params="number yaw">
 <joint name="lower_${number}_L_ball_bot" type="ball">
     <pose>
-        ${end_effector_radius*cos(yaw) - (lower_width/2)*sin(yaw)}
-        ${end_effector_radius*sin(yaw) + (lower_width/2)*cos(yaw)}
+        ${ee_radius*cos(yaw) - (lower_width/2)*sin(yaw)}
+        ${ee_radius*sin(yaw) + (lower_width/2)*cos(yaw)}
         0
         0 0 ${yaw}
     </pose>
     <parent>lower_${number}_L_link</parent>
-    <child>end_effector</child>
+    <child>ee</child>
 </joint>
 <joint name="lower_${number}_R_ball_bot" type="ball">
     <pose>
-        ${end_effector_radius*cos(yaw) + (lower_width/2)*sin(yaw)}
-        ${end_effector_radius*sin(yaw) - (lower_width/2)*cos(yaw)}
+        ${ee_radius*cos(yaw) + (lower_width/2)*sin(yaw)}
+        ${ee_radius*sin(yaw) - (lower_width/2)*cos(yaw)}
         0
         0 0 ${yaw}
     </pose>
     <parent>lower_${number}_R_link</parent>
-    <child>end_effector</child>
+    <child>ee</child>
 </joint>
 </xacro:macro>
-<xacro:joints_end_effector number="1" yaw="0"/>
-<xacro:joints_end_effector number="2" yaw="${2*pi/3}"/>
-<xacro:joints_end_effector number="3" yaw="${-2*pi/3}"/>
+<xacro:joints_ee number="1" yaw="0"/>
+<xacro:joints_ee number="2" yaw="${2*pi/3}"/>
+<xacro:joints_ee number="3" yaw="${-2*pi/3}"/>
 </robot>

File: model/delta/gazebo_links/base.sdf.xacro (robot description, xacro)
@@ -1,127 +1,6 @@
 <?xml version="1.0"?>
 <sdf xmlns:xacro="http://www.ros.org/wiki/xacro" name="base">
-<xacro:macro name="stand_part" params="number yaw">
-<visual name="stand_leg_${number}_visual_1">
-    <pose>
-        ${stand_radius*cos(yaw)}
-        ${stand_radius*sin(yaw)}
-        ${-stand_height/2}
-        0 0 ${yaw}
-    </pose>
-    <geometry><box><size>
-        ${stand_leg_depth} ${stand_leg_width} ${stand_height}
-    </size></box></geometry>
-</visual>
-<collision name="stand_leg_${number}_collision_1">
-    <pose>
-        ${stand_radius*cos(yaw)}
-        ${stand_radius*sin(yaw)}
-        ${-stand_height/2}
-        0 0 ${yaw}
-    </pose>
-    <geometry><box><size>
-        ${stand_leg_depth} ${stand_leg_depth} ${-stand_height}
-    </size></box></geometry>
-</collision>
-<inertial>
-    <pose>
-        ${stand_radius*cos(yaw)} ${stand_radius*sin(yaw)} ${-stand_height/2}
-        0 0 {yaw}
-    </pose>
-    <mass>${stand_vertical_mass}</mass>
-    <xacro:box_inertia_sdf
-        mass="${stand_vertical_mass}"
-        w="${stand_leg_depth}" h="${stand_leg_width}" d="${stand_height}"
-    />
-</inertial>
-<visual name="stand_leg_${number}_visual_2">
-    <pose>
-        ${stand_radius*cos(yaw)}
-        ${stand_radius*sin(yaw)}
-        ${-stand_height + stand_base_height/2}
-        0 0 ${yaw}
-    </pose>
-    <geometry>
-        <cylinder>
-            <length>${stand_base_height}</length>
-            <radius>${stand_base_radius}</radius>
-        </cylinder>
-    </geometry>
-</visual>
-<collision name="stand_leg_${number}_collision_2">
-    <pose>
-        ${stand_radius*cos(yaw)}
-        ${stand_radius*sin(yaw)}
-        ${-stand_height + stand_base_height/2}
-        0 0 ${yaw}
-    </pose>
-    <geometry>
-        <cylinder>
-            <length>${stand_base_height}</length>
-            <radius>${stand_base_radius}</radius>
-        </cylinder>
-    </geometry>
-    <surface>
-        <ode>
-            <mu>10</mu>
-            <mu2>10</mu2>
-            <slip>0</slip>
-            <slip2>0</slip2>
-        </ode>
-    </surface>
-</collision>
-<inertial>
-    <pose>
-        ${stand_radius*cos(yaw)} ${stand_radius*sin(yaw)} ${-stand_height+stand_base_height/2}
-        0 0 {yaw}
-    </pose>
-    <mass>${base_mass}</mass>
-    <xacro:cylinder_inertia_sdf
-        mass="${stand_base_mass}" radius="${stand_base_radius}" length="${stand_base_height}"
-    />
-</inertial>
-<visual name="stand_top_${number}_visual_3">
-    <pose>
-        ${0.5*(stand_radius+base_radius)*cos(yaw)}
-        ${0.5*(stand_radius+base_radius)*sin(yaw)}
-        0
-        0 0 ${yaw}
-    </pose>
-    <geometry><box><size>
-        ${stand_radius - base_radius}
-        ${stand_leg_width}
-        ${stand_leg_depth}
-    </size></box></geometry>
-</visual>
-<collision name="stand_leg_base_${number}_collision_3">
-    <pose>
-        ${0.5*(stand_radius+base_radius)*cos(yaw)}
-        ${0.5*(stand_radius+base_radius)*sin(yaw)}
-        0
-        0 0 ${yaw}
-    </pose>
-    <geometry><box><size>
-        ${stand_radius - base_radius}
-        ${stand_leg_width}
-        ${stand_leg_depth}
-    </size></box></geometry>
-</collision>
-<inertial>
-    <pose>
-        ${0.5*(stand_radius+base_radius)*cos(yaw)}
-        ${0.5*(stand_radius+base_radius)*sin(yaw)}
-        0
-        0 0 ${yaw}
-    </pose>
-    <xacro:box_inertia_sdf
-        mass="${stand_horizontal_mass}"
-        w="${stand_radius - base_radius}"
-        h="${stand_leg_width}"
-        d="${stand_leg_depth}"
-    />
-</inertial>
-</xacro:macro>
 <link name="base">
-<pose> 0 0 ${stand_height} 0 0 0</pose>
+<pose> 0 0 ${base_z} 0 0 0</pose>
 <visual name="base_visual">
     <geometry>
@@ -148,9 +27,4 @@
     />
 </inertial>
-<!--
-<xacro:stand_part number="1" yaw="${pi/3}"/>
-<xacro:stand_part number="2" yaw="${pi}"/>
-<xacro:stand_part number="3" yaw="${-pi/3}"/>
--->
 </link>
 </sdf>

File: model/delta/gazebo_links/end_effector.sdf.xacro (robot description, xacro)
@@ -1,9 +1,9 @@
 <?xml version="1.0"?>
 <robot xmlns:xacro="http://www.ros.org/wiki/xacro" name="delta">
-<xacro:macro name="end_effector_attachment" params="number yaw">
-<visual name="end_effector_attachment_${number}_visual">
+<xacro:macro name="ee_attachment" params="number yaw">
+<visual name="ee_attachment_${number}_visual">
     <pose>
-        ${end_effector_radius*cos(yaw)}
-        ${end_effector_radius*sin(yaw)}
+        ${ee_radius*cos(yaw)}
+        ${ee_radius*sin(yaw)}
         0
         0 ${pi/2} ${yaw + pi/2}
@@ -12,12 +12,12 @@
         <cylinder>
             <length>${lower_width}</length>
-            <radius>${end_effector_depth/2}</radius>
+            <radius>${ee_depth/2}</radius>
         </cylinder>
     </geometry>
 </visual>
-<collision name="end_effector_attachment_${number}_collision">
+<collision name="ee_attachment_${number}_collision">
     <pose>
-        ${end_effector_radius*cos(yaw)}
-        ${end_effector_radius*sin(yaw)}
+        ${ee_radius*cos(yaw)}
+        ${ee_radius*sin(yaw)}
         0
         0 ${pi/2} ${yaw + pi/2}
@@ -26,38 +26,38 @@
         <cylinder>
             <length>${lower_width}</length>
-            <radius>${end_effector_depth/2}</radius>
+            <radius>${ee_depth/2}</radius>
         </cylinder>
     </geometry>
 </collision>
 </xacro:macro>
-<link name="end_effector">
-<pose> 0 0 ${end_effector_height} 0 0 0</pose>
-<visual name="end_effector_visual">
+<link name="ee">
+<pose> 0 0 ${ee_height} 0 0 0</pose>
+<visual name="ee_visual">
     <pose>0 0 0 0 0 0</pose>
     <geometry>
         <cylinder>
-            <length>${end_effector_depth}</length>
-            <radius>${end_effector_radius}</radius>
+            <length>${ee_depth}</length>
+            <radius>${ee_radius}</radius>
         </cylinder>
     </geometry>
 </visual>
-<collision name="end_effector_collision">
+<collision name="ee_collision">
     <pose>0 0 0 0 0 0</pose>
     <geometry>
         <cylinder>
-            <length>${end_effector_depth}</length>
-            <radius>${end_effector_radius}</radius>
+            <length>${ee_depth}</length>
+            <radius>${ee_radius}</radius>
         </cylinder>
     </geometry>
 </collision>
-<xacro:end_effector_attachment number="1" yaw="0"/>
-<xacro:end_effector_attachment number="2" yaw="${2*pi/3}"/>
-<xacro:end_effector_attachment number="3" yaw="${-2*pi/3}"/>
+<xacro:ee_attachment number="1" yaw="0"/>
+<xacro:ee_attachment number="2" yaw="${2*pi/3}"/>
+<xacro:ee_attachment number="3" yaw="${-2*pi/3}"/>
 <inertial>
-    <mass>${end_effector_mass}</mass>
+    <mass>${ee_mass}</mass>
     <xacro:cylinder_inertia_sdf
-        mass="${end_effector_mass}"
-        radius="${end_effector_radius}"
-        length="${end_effector_depth}"
+        mass="${ee_mass}"
+        radius="${ee_radius}"
+        length="${ee_depth}"
     />
 </inertial>

File: model/delta/gazebo_links/lower.sdf.xacro (robot description, xacro)
@@ -7,5 +7,5 @@
     ${(base_radius + upper_length)*cos(yaw) - (lower_width/2)*sin(yaw)}
     ${(base_radius + upper_length)*sin(yaw) + (lower_width/2)*cos(yaw)}
-    ${stand_height}
+    ${base_z}
     0 ${pi - lower_inclination} ${yaw}
 </pose>
@@ -48,5 +48,5 @@
     ${(base_radius + upper_length)*cos(yaw) + (lower_width/2)*sin(yaw)}
     ${(base_radius + upper_length)*sin(yaw) - (lower_width/2)*cos(yaw)}
-    ${stand_height}
+    ${base_z}
     0 ${pi - lower_inclination} ${yaw}
 </pose>

File: model/delta/gazebo_links/upper.sdf.xacro (robot description, xacro)
@@ -4,5 +4,5 @@
 <link name="upper_${number}">
 <pose>
-    ${base_radius*cos(yaw)} ${base_radius*sin(yaw)} ${stand_height}
+    ${base_radius*cos(yaw)} ${base_radius*sin(yaw)} ${base_z}
     0 0 ${yaw}
 </pose>

File: model/delta/parameters.xacro (robot description, xacro)
@@ -1,31 +1,30 @@
 <?xml version="1.0"?>
 <robot xmlns:xacro="http://www.ros.org/wiki/xacro" name="delta_parameters">
+<!-- Properties passed as arguments -->
+<xacro:arg name="base_radius" default="0.1"/>
+<xacro:property name="base_radius" value="$(arg base_radius)" />
+<xacro:arg name="ee_radius" default="0.1"/>
+<xacro:property name="ee_radius" value="$(arg ee_radius)" />
+<xacro:arg name="upper_length" default="0.3"/>
+<xacro:property name="upper_length" value="$(arg upper_length)"/>
+<xacro:arg name="lower_length" default="0.4"/>
+<xacro:property name="lower_length" value="$(arg lower_length)"/>
+<!-- Other properties -->
 <xacro:property name="base_depth" value="0.02"/>
-<xacro:property name="base_radius" value="0.15"/>
-<xacro:property name="upper_length" value="0.3"/>
 <xacro:property name="upper_radius" value="0.005"/>
 <xacro:property name="lower_radius" value="0.005"/>
-<xacro:property name="lower_width" value="0.1"/>
-<xacro:property name="lower_length" value="0.4"/>
-<xacro:property name="end_effector_radius" value="0.1"/>
-<xacro:property name="end_effector_depth" value="0.01"/>
+<!-- Use the base radius as a sensible parallel linkage width -->
+<xacro:property name="lower_width" value="${base_radius}"/>
+<xacro:property name="ee_depth" value="0.01"/>
 <xacro:property name="base_mass" value="1"/>
 <xacro:property name="upper_mass" value="0.02"/>
 <xacro:property name="lower_mass" value="0.02"/>
-<xacro:property name="end_effector_mass" value="0.05"/>
-<xacro:property name="stand_height" value="1.1"/>
-<xacro:property name="stand_radius" value="1.2"/>
-<xacro:property name="stand_leg_width" value="0.1"/>
-<xacro:property name="stand_leg_depth" value="0.05"/>
-<xacro:property name="stand_horizontal_mass" value="0.01"/>
-<xacro:property name="stand_vertical_mass" value="0.01"/>
-<xacro:property name="stand_base_mass" value="1"/>
-<xacro:property name="stand_base_radius" value="0.12"/>
-<xacro:property name="stand_base_height" value="0.12"/>
-<xacro:property name="end_effector_height"
-    value="${stand_height - sqrt(lower_length**2 - (upper_length+base_radius-end_effector_radius)**2)}"
+<xacro:property name="ee_mass" value="0.05"/>
+<xacro:property name="base_z" value="0.8"/>
+<xacro:property name="ee_height"
+    value="${base_z - sqrt(lower_length**2 - (upper_length+base_radius-ee_radius)**2)}"
 />
 <xacro:property name="lower_inclination"
-    value="${acos((upper_length+base_radius-end_effector_radius)/lower_length)}"
+    value="${acos((upper_length+base_radius-ee_radius)/lower_length)}"
 />
 </robot>

File: model/delta/ros_joints/end_effector.urdf.xacro (robot description, xacro)
@@ -1,8 +1,8 @@
 <?xml version="1.0"?>
 <robot xmlns:xacro="http://www.ros.org/wiki/xacro" name="delta">
-<joint name="chain_1_end_to_end_effector" type="fixed">
+<joint name="chain_1_end_to_ee" type="fixed">
     <origin xyz="0 0 0" rpy="0 0 0"/>
     <parent link="chain_1_end"/>
-    <child link="end_effector"/>
+    <child link="ee"/>
 </joint>
 </robot>

File: model/delta/ros_joints/lower.urdf.xacro (robot description, xacro)
@@ -55,5 +55,5 @@
     <origin
         rpy="0 ${pi} ${number * pi * 2/3}"
-        xyz="${end_effector_radius} 0 0"
+        xyz="${ee_radius} 0 0"
     />
     <parent link="lower_${number}_end"/>

File: model/delta/ros_links/base.urdf.xacro (robot description, xacro)
@@ -3,5 +3,5 @@
 <link name="world"></link>
 <joint name="world_to_base" type="fixed">
-    <origin xyz="0 0 ${upper_length + lower_length + 4*end_effector_depth}" rpy="0 0 0"/>
+    <origin xyz="0 0 ${upper_length + lower_length + 4*ee_depth}" rpy="0 0 0"/>
     <parent link="world"/>
     <child link="base"/>

File: model/delta/ros_links/end_effector.urdf.xacro (robot description, xacro)
@@ -1,20 +1,20 @@
 <?xml version="1.0"?>
 <robot xmlns:xacro="http://www.ros.org/wiki/xacro" name="delta">
-<link name="end_effector">
+<link name="ee">
 <visual>
     <geometry>
         <cylinder
-            length="${end_effector_depth}"
-            radius="${end_effector_radius}"
+            length="${ee_depth}"
+            radius="${ee_radius}"
         />
     </geometry>
     <origin rpy="0 0 0" xyz="0 0 0"/>
-    <material name="end_effector"/>
+    <material name="ee"/>
 </visual>
 <collision>
     <geometry>
         <cylinder
-            length="${end_effector_depth}"
-            radius="${end_effector_radius}"
+            length="${ee_depth}"
+            radius="${ee_radius}"
         />
     </geometry>
@@ -23,40 +23,40 @@
 <visual>
     <geometry>
-        <cylinder length="${lower_width}" radius="${end_effector_depth/2}" />
+        <cylinder length="${lower_width}" radius="${ee_depth/2}" />
     </geometry>
-    <origin xyz="${end_effector_radius} 0 0" rpy="0 ${pi/2} ${pi/2}" />
-    <material name="end_effector"/>
+    <origin xyz="${ee_radius} 0 0" rpy="0 ${pi/2} ${pi/2}" />
+    <material name="ee"/>
 </visual>
 <collision>
     <geometry>
-        <cylinder length="${lower_width}" radius="${end_effector_depth/2}" />
+        <cylinder length="${lower_width}" radius="${ee_depth/2}" />
     </geometry>
-    <origin xyz="${end_effector_radius} 0 0" rpy="0 ${pi/2} ${pi/2}" />
+    <origin xyz="${ee_radius} 0 0" rpy="0 ${pi/2} ${pi/2}" />
 </collision>
 <visual>
     <geometry>
-        <cylinder length="${lower_width}" radius="${end_effector_depth/2}" />
+        <cylinder length="${lower_width}" radius="${ee_depth/2}" />
     </geometry>
-    <origin xyz="${cos(pi*2/3)*end_effector_radius} ${sin(pi*2/3)*end_effector_radius} 0" rpy="0 ${pi/2} ${pi*7/6}" />
-    <material name="end_effector"/>
+    <origin xyz="${cos(pi*2/3)*ee_radius} ${sin(pi*2/3)*ee_radius} 0" rpy="0 ${pi/2} ${pi*7/6}" />
+    <material name="ee"/>
 </visual>
 <collision>
     <geometry>
-        <cylinder length="${lower_width}" radius="${end_effector_depth/2}" />
+        <cylinder length="${lower_width}" radius="${ee_depth/2}" />
     </geometry>
-    <origin xyz="${cos(pi*2/3)*end_effector_radius} ${sin(pi*2/3)*end_effector_radius} 0" rpy="0 ${pi/2} ${pi*7/6}" />
+    <origin xyz="${cos(pi*2/3)*ee_radius} ${sin(pi*2/3)*ee_radius} 0" rpy="0 ${pi/2} ${pi*7/6}" />
 </collision>
 <visual>
     <geometry>
-        <cylinder length="${lower_width}" radius="${end_effector_depth/2}" />
+        <cylinder length="${lower_width}" radius="${ee_depth/2}" />
     </geometry>
-    <origin xyz="${cos(pi*4/3)*end_effector_radius} ${sin(pi*4/3)*end_effector_radius} 0" rpy="0 ${pi/2} ${pi*11/6}" />
-    <material name="end_effector"/>
+    <origin xyz="${cos(pi*4/3)*ee_radius} ${sin(pi*4/3)*ee_radius} 0" rpy="0 ${pi/2} ${pi*11/6}" />
+    <material name="ee"/>
 </visual>
 <collision>
     <geometry>
-        <cylinder length="${lower_width}" radius="${end_effector_depth/2}" />
+        <cylinder length="${lower_width}" radius="${ee_depth/2}" />
     </geometry>
-    <origin xyz="${cos(pi*4/3)*end_effector_radius} ${sin(pi*4/3)*end_effector_radius} 0" rpy="0 ${pi/2} ${pi*11/6}" />
+    <origin xyz="${cos(pi*4/3)*ee_radius} ${sin(pi*4/3)*ee_radius} 0" rpy="0 ${pi/2} ${pi*11/6}" />
 </collision>
 </link>
