Commit message: Added gripper to delta

File: model/delta/gazebo_joints/end_effector.sdf.xacro (robot description, xacro)
@@ -26,3 +26,48 @@
 <xacro:joints_ee number="2" yaw="${2*pi/3}"/>
 <xacro:joints_ee number="3" yaw="${-2*pi/3}"/>
+<joint name="theta_4" type="revolute">
+    <pose>0 0 0 0 0 0</pose>
+    <parent>ee</parent>
+    <child>gripper_base</child>
+    <axis>
+        <xyz>0 0 1</xyz>
+        <limit>
+            <lower>${-pi*0.99}</lower>
+            <upper>${pi*0.99}</upper>
+            <velocity>100</velocity>
+        </limit>
+    </axis>
+</joint>
+<joint name="gripper" type="revolute">
+    <pose>0 0 0 0 0 0</pose>
+    <parent>gripper_base</parent>
+    <child>gripper_left</child>
+    <axis>
+        <xyz>1 0 0</xyz>
+        <limit>
+            <lower>0</lower>
+            <upper>${pi/2}</upper>
+            <velocity>100</velocity>
+        </limit>
+    </axis>
+</joint>
+<joint name="gripper_mimic" type="revolute">
+    <pose>0 0 0 0 0 0</pose>
+    <parent>gripper_base</parent>
+    <child>gripper_right</child>
+    <axis>
+        <xyz>-1 0 0</xyz>
+        <limit>
+            <lower>0</lower>
+            <upper>${pi/2}</upper>
+            <velocity>100</velocity>
+        </limit>
+    </axis>
+</joint>
+<plugin name="gripper_mimic_joint_plugin" filename="libroboticsgroup_gazebo_mimic_joint_plugin.so">
+  <joint>gripper</joint>
+  <mimicJoint>gripper_mimic</mimicJoint>
+  <multiplier>1</multiplier>
+</plugin>
+    -->
 </robot>

File: model/delta/gazebo_links/end_effector.sdf.xacro (robot description, xacro)
@@ -63,3 +63,87 @@
 </inertial>
 </link>
+<link name="gripper_base">
+<pose> 0 0 ${ee_height} 0 0 0</pose>
+<visual name="gripper_base_visual">
+    <pose>0 0 -0.04 0 0 0</pose>
+    <geometry>
+        <box>
+            <size>0.05 0.1 0.08</size>
+        </box>
+    </geometry>
+</visual>
+<collision name="gripper_base_collision">
+    <pose>0 0 -0.04 0 0 0</pose>
+    <geometry>
+        <box>
+            <size>0.05 0.1 0.08</size>
+        </box>
+    </geometry>
+</collision>
+<inertial>
+    <mass>${ee_mass/10}</mass>
+    <xacro:box_inertia_sdf
+        mass="${ee_mass/10}"
+        w="0.05"
+        h="0.1"
+        d="0.08"
+    />
+</inertial>
+</link>
+<link name="gripper_left">
+<pose> 0 -0.05 ${ee_height-0.08} 0 0 0</pose>
+<visual name="gripper_left_visual">
+    <pose>0 0 -0.05 0 0 0</pose>
+    <geometry>
+        <box>
+            <size>0.05 0.005 0.1</size>
+        </box>
+    </geometry>
+</visual>
+<collision name="gripper_left_collision">
+    <pose>0 0 -0.05 0 0 0</pose>
+    <geometry>
+        <box>
+            <size>0.05 0.005 0.1</size>
+        </box>
+    </geometry>
+</collision>
+<inertial>
+    <mass>${ee_mass/10}</mass>
+    <xacro:box_inertia_sdf
+        mass="${ee_mass/10}"
+        w="0.05"
+        h="0.005"
+        d="0.1"
+    />
+</inertial>
+</link>
+<link name="gripper_right">
+<pose> 0 0.05 ${ee_height-0.08} 0 0 0</pose>
+<visual name="gripper_right_visual">
+    <pose>0 0 -0.05 0 0 0</pose>
+    <geometry>
+        <box>
+            <size>0.05 0.005 0.1</size>
+        </box>
+    </geometry>
+</visual>
+<collision name="gripper_right_collision">
+    <pose>0 0 -0.05 0 0 0</pose>
+    <geometry>
+        <box>
+            <size>0.05 0.005 0.1</size>
+        </box>
+    </geometry>
+</collision>
+<inertial>
+    <mass>${ee_mass/10}</mass>
+    <xacro:box_inertia_sdf
+        mass="${ee_mass/10}"
+        w="0.05"
+        h="0.005"
+        d="0.1"
+    />
+</inertial>
+</link>
 </robot>

File: model/delta/ros_joints/end_effector.urdf.xacro (robot description, xacro)
@@ -6,3 +6,60 @@
     <child link="ee"/>
 </joint>
+<joint name="theta_4" type="revolute">
+    <origin xyz="0 0 0" rpy="0 0 0"/>
+    <parent link="ee"/>
+    <child link="gripper_base"/>
+    <axis xyz="0 0 1"/>
+    <limit
+        effort="1000.0"
+        lower="${-pi*0.99}"
+        upper="${pi*0.99}"
+        velocity="5"
+    />
+</joint>
+<joint name="gripper" type="revolute">
+    <origin xyz="0 -0.05 -0.08" rpy="0 0 0"/>
+    <parent link="gripper_base"/>
+    <child link="gripper_left"/>
+    <axis xyz="1 0 0"/>
+    <limit
+        effort="1000.0"
+        lower="0"
+        upper="${pi/2}"
+        velocity="5"
+    />
+</joint>
+<joint name="gripper_mimic" type="revolute">
+    <origin xyz="0 0.05 -0.08" rpy="0 0 0"/>
+    <parent link="gripper_base"/>
+    <child link="gripper_right"/>
+    <axis xyz="-1 0 0"/>
+    <limit
+        effort="1000.0"
+        lower="0"
+        upper="${pi/2}"
+        velocity="5"
+    />
+    <mimic joint="gripper"/>
+</joint>
+<transmission name="theta_4_tran">
+    <type>transmission_interface/SimpleTransmission</type>
+    <joint name="theta_4">
+        <hardwareInterface>hardware_interface/PositionJointInterface</hardwareInterface>
+    </joint>
+    <actuator name="theta_4">
+        <hardwareInterface>hardware_interface/PositionJointInterface</hardwareInterface>
+        <mechanicalReduction>1</mechanicalReduction>
+    </actuator>
+</transmission>
+<transmission name="gripper_tran">
+    <type>transmission_interface/SimpleTransmission</type>
+    <joint name="gripper">
+        <hardwareInterface>hardware_interface/PositionJointInterface</hardwareInterface>
+    </joint>
+    <actuator name="gripper">
+        <hardwareInterface>hardware_interface/PositionJointInterface</hardwareInterface>
+        <mechanicalReduction>1</mechanicalReduction>
+    </actuator>
+</transmission>
 </robot>

File: model/delta/ros_joints/upper.urdf.xacro (robot description, xacro)
@@ -15,5 +15,5 @@
         xyz="${cos(yaw)*base_radius} ${sin(yaw)*base_radius} 0"
     />
-    <parent link="base"/>
+    <parent link="base_link"/>
     <child link="upper_${number}"/>
 </joint>

File: model/delta/ros_links/base.urdf.xacro (robot description, xacro)
@@ -5,7 +5,7 @@
     <origin xyz="0 0 ${upper_length + lower_length + 4*ee_depth}" rpy="0 0 0"/>
     <parent link="world"/>
-    <child link="base"/>
+    <child link="base_link"/>
 </joint>
-<link name="base">
+<link name="base_link">
 <visual>
     <geometry>

File: model/delta/ros_links/end_effector.urdf.xacro (robot description, xacro)
@@ -61,3 +61,45 @@
 </collision>
 </link>
+<link name="gripper_base">
+<visual>
+    <geometry>
+        <box size="0.05 0.1 0.08"/>
+    </geometry>
+    <origin xyz="0 0 -0.04"/>
+</visual>
+<collision>
+    <geometry>
+        <box size="0.05 0.1 0.08"/>
+    </geometry>
+    <origin xyz="0 0 -0.04"/>
+</collision>
+</link>
+<link name="gripper_left">
+<visual>
+    <geometry>
+        <box size="0.05 0.005 0.1"/>
+    </geometry>
+    <origin xyz="0 0 -0.05"/>
+</visual>
+<collision>
+    <geometry>
+        <box size="0.05 0.005 0.1"/>
+    </geometry>
+    <origin xyz="0 0 -0.05"/>
+</collision>
+</link>
+<link name="gripper_right">
+<visual>
+    <geometry>
+        <box size="0.05 0.005 0.1"/>
+    </geometry>
+    <origin xyz="0 0 -0.05"/>
+</visual>
+<collision>
+    <geometry>
+        <box size="0.05 0.005 0.1"/>
+    </geometry>
+    <origin xyz="0 0 -0.05"/>
+</collision>
+</link>
 </robot>
