Commit message: Gripper control working better now, but still can't get gazebo mimic plugin to work.

File: model/delta/gazebo.sdf.xacro (robot description, xacro)
@@ -18,4 +18,23 @@
 <xacro:include filename="gazebo_joints/end_effector.sdf.xacro"/>
 <plugin name="gazebo_ros_control" filename="libgazebo_ros_control.so"/>
+<xacro:macro name="mimic_joint_plugin_gazebo" params="name_prefix parent_joint mimic_joint has_pid:=false multiplier:=1.0 offset:=0 sensitiveness:=0.0 max_effort:=1.0 robot_namespace:=''">
+  <plugin name="${name_prefix}mimic_joint_plugin" filename="libroboticsgroup_gazebo_mimic_joint_plugin.so">
+    <joint>${parent_joint}</joint>
+    <mimicJoint>${mimic_joint}</mimicJoint>
+    <xacro:if value="${has_pid}">                     <!-- if set to true, PID parameters from "/gazebo_ros_control/pid_gains/${mimic_joint}" are loaded -->
+      <hasPID />
+    </xacro:if>
+    <multiplier>${multiplier}</multiplier>
+    <offset>${offset}</offset>
+    <sensitiveness>${sensitiveness}</sensitiveness>   <!-- if absolute difference between setpoint and process value is below this threshold, do nothing; 0.0 = disable [rad] -->
+    <maxEffort>${max_effort}</maxEffort>              <!-- only taken into account if has_pid:=true [Nm] -->
+    <xacro:unless value="${robot_namespace == ''}">
+      <robotNamespace>${robot_namespace}</robotNamespace>
+    </xacro:unless>
+  </plugin>
+</xacro:macro>
+<xacro:mimic_joint_plugin_gazebo name_prefix="gripper"
+  parent_joint="gripper" mimic_joint="gripper_mimic"
+  has_pid="true" multiplier="1.0" max_effort="10.0" />
 </model>
 </sdf>

File: model/delta/gazebo_joints/end_effector.sdf.xacro (robot description, xacro)
@@ -40,9 +40,9 @@
 </joint>
 <joint name="gripper" type="revolute">
-    <pose>0 0 0 0 0 0</pose>
+    <pose>0 0 0 0.6 0 0</pose>
     <parent>gripper_base</parent>
     <child>gripper_left</child>
     <axis>
-        <xyz>1 0 0</xyz>
+        <xyz>-1 0 0</xyz>
         <limit>
             <lower>0</lower>
@@ -57,5 +57,5 @@
     <child>gripper_right</child>
     <axis>
-        <xyz>-1 0 0</xyz>
+        <xyz>1 0 0</xyz>
         <limit>
             <lower>0</lower>
@@ -65,9 +65,3 @@
     </axis>
 </joint>
-<plugin name="gripper_mimic_joint_plugin" filename="libroboticsgroup_gazebo_mimic_joint_plugin.so">
-  <joint>gripper</joint>
-  <mimicJoint>gripper_mimic</mimicJoint>
-  <multiplier>1</multiplier>
-</plugin>
-    -->
 </robot>

File: model/delta/gazebo_links/end_effector.sdf.xacro (robot description, xacro)
@@ -92,5 +92,5 @@
 </link>
 <link name="gripper_left">
-<pose> 0 -0.05 ${ee_height-0.08} 0 0 0</pose>
+<pose> 0 -0.05 ${ee_height-0.08} 0.6 0 0</pose>
 <visual name="gripper_left_visual">
     <pose>0 0 -0.05 0 0 0</pose>
@@ -120,5 +120,5 @@
 </link>
 <link name="gripper_right">
-<pose> 0 0.05 ${ee_height-0.08} 0 0 0</pose>
+<pose> 0 0.05 ${ee_height-0.08} -0.6 0 0</pose>
 <visual name="gripper_right_visual">
     <pose>0 0 -0.05 0 0 0</pose>

File: model/delta/ros_joints/end_effector.urdf.xacro (robot description, xacro)
@@ -19,8 +19,8 @@
 </joint>
 <joint name="gripper" type="revolute">
-    <origin xyz="0 -0.05 -0.08" rpy="0 0 0"/>
+    <origin xyz="0 -0.05 -0.08" rpy="0.6 0 0"/>
     <parent link="gripper_base"/>
     <child link="gripper_left"/>
-    <axis xyz="1 0 0"/>
+    <axis xyz="-1 0 0"/>
     <limit
         effort="1000.0"
@@ -31,8 +31,8 @@
 </joint>
 <joint name="gripper_mimic" type="revolute">
-    <origin xyz="0 0.05 -0.08" rpy="0 0 0"/>
+    <origin xyz="0 0.05 -0.08" rpy="-0.6 0 0"/>
     <parent link="gripper_base"/>
     <child link="gripper_right"/>
-    <axis xyz="-1 0 0"/>
+    <axis xyz="1 0 0"/>
     <limit
         effort="1000.0"

Commit message: Fixed gripper in delta simulation

File: model/delta/gazebo.sdf.xacro (robot description, xacro)
@@ -18,23 +18,10 @@
 <xacro:include filename="gazebo_joints/end_effector.sdf.xacro"/>
 <plugin name="gazebo_ros_control" filename="libgazebo_ros_control.so"/>
-<xacro:macro name="mimic_joint_plugin_gazebo" params="name_prefix parent_joint mimic_joint has_pid:=false multiplier:=1.0 offset:=0 sensitiveness:=0.0 max_effort:=1.0 robot_namespace:=''">
-  <plugin name="${name_prefix}mimic_joint_plugin" filename="libroboticsgroup_gazebo_mimic_joint_plugin.so">
-    <joint>${parent_joint}</joint>
-    <mimicJoint>${mimic_joint}</mimicJoint>
-    <xacro:if value="${has_pid}">                     <!-- if set to true, PID parameters from "/gazebo_ros_control/pid_gains/${mimic_joint}" are loaded -->
-      <hasPID />
-    </xacro:if>
-    <multiplier>${multiplier}</multiplier>
-    <offset>${offset}</offset>
-    <sensitiveness>${sensitiveness}</sensitiveness>   <!-- if absolute difference between setpoint and process value is below this threshold, do nothing; 0.0 = disable [rad] -->
-    <maxEffort>${max_effort}</maxEffort>              <!-- only taken into account if has_pid:=true [Nm] -->
-    <xacro:unless value="${robot_namespace == ''}">
-      <robotNamespace>${robot_namespace}</robotNamespace>
-    </xacro:unless>
-  </plugin>
-</xacro:macro>
-<xacro:mimic_joint_plugin_gazebo name_prefix="gripper"
-  parent_joint="gripper" mimic_joint="gripper_mimic"
-  has_pid="true" multiplier="1.0" max_effort="10.0" />
+<plugin name="gripper_mimic_joint_plugin" filename="libroboticsgroup_upatras_gazebo_mimic_joint_plugin.so">
+    <joint>gripper</joint>
+    <mimicJoint>gripper_mimic</mimicJoint>
+    <hasPID />
+    <maxEffort>5000</maxEffort>
+</plugin>
 </model>
 </sdf>

File: model/delta/gazebo_joints/end_effector.sdf.xacro (robot description, xacro)
@@ -40,5 +40,5 @@
 </joint>
 <joint name="gripper" type="revolute">
-    <pose>0 0 0 0.6 0 0</pose>
+    <pose> 0 0 0 0 0 0</pose>
     <parent>gripper_base</parent>
     <child>gripper_left</child>
@@ -53,5 +53,5 @@
 </joint>
 <joint name="gripper_mimic" type="revolute">
-    <pose>0 0 0 0 0 0</pose>
+    <pose> 0 0 0 0 0 0</pose>
     <parent>gripper_base</parent>
     <child>gripper_right</child>

File: model/delta/gazebo_links/end_effector.sdf.xacro (robot description, xacro)
@@ -66,82 +66,85 @@
 <pose> 0 0 ${ee_height} 0 0 0</pose>
 <visual name="gripper_base_visual">
-    <pose>0 0 -0.04 0 0 0</pose>
+    <pose>0 0 -0.025 0 0 0</pose>
     <geometry>
         <box>
-            <size>0.05 0.1 0.08</size>
+            <size>0.03 0.05 0.05</size>
         </box>
     </geometry>
 </visual>
 <collision name="gripper_base_collision">
-    <pose>0 0 -0.04 0 0 0</pose>
+    <pose>0 0 -0.025 0 0 0</pose>
     <geometry>
         <box>
-            <size>0.05 0.1 0.08</size>
+            <size>0.03 0.05 0.05</size>
         </box>
     </geometry>
 </collision>
 <inertial>
-    <mass>${ee_mass/10}</mass>
+    <pose>0 0 -0.025 0 0 0</pose>
+    <mass>${ee_mass}</mass>
     <xacro:box_inertia_sdf
-        mass="${ee_mass/10}"
-        w="0.05"
-        h="0.1"
-        d="0.08"
+        mass="${ee_mass}"
+        w="0.03"
+        h="0.05"
+        d="0.05"
     />
 </inertial>
 </link>
 <link name="gripper_left">
-<pose> 0 -0.05 ${ee_height-0.08} 0.6 0 0</pose>
+<pose> 0 -0.025 ${ee_height-0.05} 0.4 0 0</pose>
 <visual name="gripper_left_visual">
-    <pose>0 0 -0.05 0 0 0</pose>
+    <pose>0 0 -0.025 0 0 0</pose>
     <geometry>
         <box>
-            <size>0.05 0.005 0.1</size>
+            <size>0.03 0.005 0.05</size>
         </box>
     </geometry>
 </visual>
 <collision name="gripper_left_collision">
-    <pose>0 0 -0.05 0 0 0</pose>
+    <pose>0 0 -0.025 0 0 0</pose>
     <geometry>
         <box>
-            <size>0.05 0.005 0.1</size>
+            <size>0.03 0.005 0.05</size>
         </box>
     </geometry>
 </collision>
 <inertial>
-    <mass>${ee_mass/10}</mass>
+    <pose>0 0 -0.025 0 0 0</pose>
+    <mass>${ee_mass}</mass>
     <xacro:box_inertia_sdf
-        mass="${ee_mass/10}"
-        w="0.05"
+        mass="${ee_mass}"
+        w="0.03"
         h="0.005"
-        d="0.1"
+        d="0.05"
     />
 </inertial>
 </link>
 <link name="gripper_right">
-<pose> 0 0.05 ${ee_height-0.08} -0.6 0 0</pose>
+<pose> 0 0.025 ${ee_height-0.05} -0.4 0 0</pose>
 <visual name="gripper_right_visual">
-    <pose>0 0 -0.05 0 0 0</pose>
+    <pose>0 0 -0.025 0 0 0</pose>
     <geometry>
         <box>
-            <size>0.05 0.005 0.1</size>
+            <size>0.03 0.005 0.05</size>
         </box>
     </geometry>
 </visual>
 <collision name="gripper_right_collision">
-    <pose>0 0 -0.05 0 0 0</pose>
+    <pose>0 0 -0.025 0 0 0</pose>
     <geometry>
         <box>
-            <size>0.05 0.005 0.1</size>
+            <size>0.03 0.005 0.05</size>
         </box>
     </geometry>
 </collision>
 <inertial>
-    <mass>${ee_mass/10}</mass>
+    <pose>0 0 -0.025 0 0 0</pose>
+    <mass>${ee_mass}</mass>
     <xacro:box_inertia_sdf
-        mass="${ee_mass/10}"
-        w="0.05"
+        mass="${ee_mass}"
+        w="0.03"
         h="0.005"
-        d="0.1"
+        d="0.05"
     />
 </inertial>

Commit message: Editted delta model so it can pick up a block.

File: model/delta/gazebo.sdf.xacro (robot description, xacro)
@@ -2,5 +2,4 @@
 <sdf version='1.4' xmlns:xacro="http://www.ros.org/wiki/xacro">
 <model name="delta">
-<selfCollide>true</selfCollide>
 <joint name="world_fix" type="fixed">
     <pose>0 0 0 0 0 0</pose>

File: model/delta/gazebo_links/end_effector.sdf.xacro (robot description, xacro)
@@ -109,4 +109,18 @@
         </box>
     </geometry>
+    <surface>
+        <contact>
+            <ode>
+                <kp>1e15</kp>
+                <kd>1e13</kd>
+            </ode>
+        </contact>
+        <friction>
+            <ode>
+                <mu>1</mu>
+                <mu2>1</mu2>
+            </ode>
+        </friction>
+    </surface>
 </collision>
 <inertial>
@@ -138,4 +152,18 @@
         </box>
     </geometry>
+    <surface>
+        <contact>
+            <ode>
+                <kp>1e15</kp>
+                <kd>1e13</kd>
+            </ode>
+        </contact>
+        <friction>
+            <ode>
+                <mu>1</mu>
+                <mu2>1</mu2>
+            </ode>
+        </friction>
+    </surface>
 </collision>
 <inertial>

File: model/delta/materials.urdf.xacro (robot description, xacro)
@@ -5,11 +5,11 @@
 </material>
 <material name="upper">
+    <color rgba="1 0 1 1"/>
+</material>
+<material name="lower">
+    <color rgba="0 0 1 1"/>
+</material>
+<material name="ee">
     <color rgba="0 1 1 1"/>
 </material>
-<material name="lower">
-    <color rgba="0 1 0 1"/>
-</material>
-<material name="ee">
-    <color rgba="1 0 1 1"/>
-</material>
 </robot>

File: model/delta/parameters.xacro (robot description, xacro)
@@ -21,5 +21,5 @@
 <xacro:property name="lower_mass" value="0.02"/>
 <xacro:property name="ee_mass" value="0.05"/>
-<xacro:property name="base_z" value="0.8"/>
+<xacro:property name="base_z" value="0.45"/>
 <xacro:property name="ee_height"
     value="${base_z - sqrt(lower_length**2 - (upper_length+base_radius-ee_radius)**2)}"

File: model/delta/ros_links/end_effector.urdf.xacro (robot description, xacro)
@@ -67,4 +67,5 @@
     </geometry>
     <origin xyz="0 0 -0.025" rpy="0 0 0"/>
+    <material name="ee"/>
 </visual>
 <collision>
@@ -81,4 +82,5 @@
     </geometry>
     <origin xyz="0 0 -0.025"/>
+    <material name="ee"/>
 </visual>
 <collision>
@@ -95,4 +97,5 @@
     </geometry>
     <origin xyz="0 0 -0.025"/>
+    <material name="ee"/>
 </visual>
 <collision>
