Commit message: More editing of serial model for simulation.

File: model/delta/ros_links/end_effector.urdf.xacro (robot description, xacro)
@@ -89,4 +89,18 @@
     </geometry>
     <origin xyz="0 0 -0.025"/>
+    <surface>
+        <contact>
+            <ode>
+                <kp>1e15</kp>
+                <kd>1e13</kd>
+            </ode>
+        </contact>
+        <friction>
+            <ode>
+                <mu>1</mu>
+                <mu2>1</mu2>
+            </ode>
+        </friction>
+    </surface>
 </collision>
 </link>
@@ -104,4 +118,18 @@
     </geometry>
     <origin xyz="0 0 -0.025"/>
+    <surface>
+        <contact>
+            <ode>
+                <kp>1e15</kp>
+                <kd>1e13</kd>
+            </ode>
+        </contact>
+        <friction>
+            <ode>
+                <mu>1</mu>
+                <mu2>1</mu2>
+            </ode>
+        </friction>
+    </surface>
 </collision>
 </link>

File: model/serial/ros2.urdf.xacro (robot description, xacro)
@@ -25,9 +25,4 @@
 <link name="${link}">
 <xacro:if value="${a!=0}">
-<inertial>
-    <origin rpy="0 ${pi/2} 0" xyz="${a/2} 0 0"/>
-    <mass value="${ma}"/>
-    <xacro:cylinder_inertia_urdf mass="${ma}" radius="${ra}" length="${a}"/>
-</inertial>
 <visual>
     <geometry>
@@ -45,9 +40,4 @@
 </xacro:if>
 <xacro:if value="${d!=0}">
-<inertial>
-    <origin rpy="0 0 0" xyz="0 0 ${-d/2}"/>
-    <mass value="${md}"/>
-    <xacro:cylinder_inertia_urdf mass="${md}" radius="${rd}" length="${d}"/>
-</inertial>
 <visual>
     <geometry>
@@ -65,4 +55,13 @@
 </collision>
 </xacro:if>
+<inertial>
+    <origin rpy="0 0 0" xyz="0 0 0"/>
+    <mass value="${ma+md}"/>
+    <inertia
+        ixx="${ma*(ra**2)/2 + md*(rd**2)/4 + md*(d**2)/3}"
+        iyy="${ma*(ra**2)/4 + ma*(a**2)/3 + md*(rd**2)/4 + md*(d**2)/3}"
+        izz="${md*(rd**2)/2 + ma*(ra**2)/4 + ma*(a**2)/3}"
+        ixy="0" ixz="0" iyz="0"/>
+</inertial>
 </link>
 </xacro:macro>
@@ -76,5 +75,5 @@
 <link name="base_link"/>
 <joint name="base_joint" type="fixed">
-    <origin rpy="0 0 0" xyz="0 0 0"/>
+    <origin rpy="0 0 0" xyz="0 0 ${0.1*d1}"/>
     <parent link="base_link"/>
     <child link="fixed_base"/>
@@ -82,5 +81,5 @@
 <link name="fixed_base">
 <inertial>
-    <origin rpy="0 0 0" xyz="0 0 ${0.05*d1}"/>
+    <origin rpy="0 0 0" xyz="0 0 ${-0.05*d1}"/>
     <mass value="${md1}"/>
     <xacro:cylinder_inertia_urdf mass="${md1}" radius="${rd1}" length="${0.1*d1}"/>
@@ -90,5 +89,5 @@
         <cylinder length="${0.1*d1}" radius="${rd1}"/>
     </geometry>
-    <origin rpy="0 0 0" xyz="0 0 ${0.05*d1}"/>
+    <origin rpy="0 0 0" xyz="0 0 ${-0.05*d1}"/>
     <material name="mat1"/>
 </visual>
@@ -97,9 +96,9 @@
         <cylinder length="${0.1*d1}" radius="${rd1}"/>
     </geometry>
-    <origin rpy="0 0 0" xyz="0 0 ${0.05*d1}"/>
+    <origin rpy="0 0 0" xyz="0 0 ${-0.05*d1}"/>
 </collision>
 </link>
 <xacro:arm_link joint="theta_1" parent="fixed_base" link="link1"
-    a_prev="0" alpha="${alpha1}" d="${d1}" a="${a1}" theta="${theta1}" ra="${ra1}" ma="${ma1}" rd="${rd1}" md="${md1}" material="mat1"
+    a_prev="0" alpha="${alpha1}" d="${0.9*d1}" a="${a1}" theta="${theta1}" ra="${ra1}" ma="${ma1}" rd="${rd1}" md="${md1}" material="mat1"
 />
 <xacro:arm_link joint="theta_2" parent="link1" link="link2"
@@ -131,9 +130,25 @@
     </geometry>
     <origin xyz="0 0 0.025"/>
-</collision>
-<inertial>
-    <origin xyz="0 0 0.025"/>
-    <mass value="${ma6/5}"/>
-    <xacro:box_inertia_urdf mass="${ma6}" w="0.02" h="0.01" d="0.05"/>
+    <gazebo>
+    <surface>
+        <contact>
+            <ode>
+                <kp>1e15</kp>
+                <kd>1e13</kd>
+            </ode>
+        </contact>
+        <friction>
+            <ode>
+                <mu>1</mu>
+                <mu2>1</mu2>
+            </ode>
+        </friction>
+    </surface>
+    </gazebo>
+</collision>
+<inertial>
+    <origin xyz="0 0 0.025"/>
+    <mass value="${ma6*2}"/>
+    <xacro:box_inertia_urdf mass="${ma6*2}" w="0.02" h="0.01" d="0.05"/>
 </inertial>
 </link>
@@ -151,9 +166,25 @@
     </geometry>
     <origin xyz="0 0 0.025"/>
-</collision>
-<inertial>
-    <origin xyz="0 0 0.025"/>
-    <mass value="${ma6/5}"/>
-    <xacro:box_inertia_urdf mass="${ma6}" w="0.02" h="0.01" d="0.05"/>
+    <gazebo>
+    <surface>
+        <contact>
+            <ode>
+                <kp>1e15</kp>
+                <kd>1e13</kd>
+            </ode>
+        </contact>
+        <friction>
+            <ode>
+                <mu>1</mu>
+                <mu2>1</mu2>
+            </ode>
+        </friction>
+    </surface>
+    </gazebo>
+</collision>
+<inertial>
+    <origin xyz="0 0 0.025"/>
+    <mass value="${ma6*2}"/>
+    <xacro:box_inertia_urdf mass="${ma6*2}" w="0.02" h="0.01" d="0.05"/>
 </inertial>
 </link>
@@ -195,4 +226,10 @@
 <gazebo>
     <plugin name="gazebo_ros_control" filename="libgazebo_ros_control.so"/>
+    <plugin name="gripper_mimic_joint_plugin" filename="libroboticsgroup_upatras_gazebo_mimic_joint_plugin.so">
+        <joint>gripper</joint>
+        <mimicJoint>gripper_mimic</mimicJoint>
+        <hasPID />
+        <maxEffort>5000</maxEffort>
+    </plugin>
 </gazebo>
 </robot>
